File: Interface.kicad_pcb (KiCad board)
At the start: 2 copper layers, 36 x 25 mm, 20 parts, among them IC1 PI6CG18201ZDIEX, J1 Conn_01x07_MountingPin, J2 PCI_Express_x1 female connect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, U1 AMS1117-1.8, Y1 25MHz

Commit message: Continue layout
Parts:
- added H1: MountingHole, MountingHole:MountingHole_3.2mm_M3_ISO7380, B.Cu at (102.5, 77.5)
- added H2: MountingHole, MountingHole:MountingHole_3.2mm_M3_ISO7380, F.Cu at (136.0, 82.5)
- added J3: Conn_01x07_MountingPin, Connector_Molex:Molex_PicoBlade_53048-0710_1x07_P1.25mm_Horizontal, F.Cu at (131.5, 87.8)
- added TP1: 12V, TestPoint:TestPoint_THTPad_D1.0mm_Drill0.5mm, F.Cu at (131.5, 77.2)
Connections:
- J2 pad A2: unconnected-(J2-+12V-PadA2) -> /12V
- J2 pad A3: unconnected-(J2-+12V-PadA2) -> /12V
- J2 pad B1: unconnected-(J2-+12V-PadA2) -> /12V
- J2 pad B2: unconnected-(J2-+12V-PadA2) -> /12V
- J2 pad B3: unconnected-(J2-+12V-PadA2) -> /12V
Routing:
- net GND: track 42.9 -> 56.2 mm, vias 16 -> 18
- net unconnected-(J2-+12V-PadA2): track 8.74 -> 0.00 mm
- net /3V3: track 73.1 -> 70.6 mm
- net /Rx-: track 20.5 -> 21.3 mm
- net /Rx+: track 21.7 -> 22.5 mm
- net /Tx+: track 22.0 -> 22.5 mm
- net /12V: vias 0 -> 2
- added copper zone on B.Cu, net /12V
- added copper zone on F.Cu, net /12V
Other:
- outline, holes or cut-outs redrawn
- board text added: "GND GND Tx+ Tx- Rx+ Rx- 3V3"
- board text added: "PCIe clock injector"

Commit message: Layout finished
Parts:
- removed H2: MountingHole, MountingHole:MountingHole_3.2mm_M3_ISO7380
- removed J3: Conn_01x07_MountingPin, Connector_Molex:Molex_PicoBlade_53048-0710_1x07_P1.25mm_Horizontal
- added R4: 0, Resistor_SMD:R_0402_1005Metric_Pad0.72x0.64mm_HandSolder, F.Cu at (126.0, 90.1)
- added R5: 0, Resistor_SMD:R_0402_1005Metric_Pad0.72x0.64mm_HandSolder, F.Cu at (126.0, 90.9)
- added R6: 0, Resistor_SMD:R_0402_1005Metric_Pad0.72x0.64mm_HandSolder, F.Cu at (128.4, 80.1)
- added R7: 0, Resistor_SMD:R_0402_1005Metric_Pad0.72x0.64mm_HandSolder, F.Cu at (129.2, 80.1)
- added REF**: KiCad-Logo_5mm_SilkScreen, Symbol:KiCad-Logo_5mm_SilkScreen, B.Cu at (123.2, 91.2)
- added REF**: OSHW-Symbol_6.7x6mm_SilkScreen, Symbol:OSHW-Symbol_6.7x6mm_SilkScreen, B.Cu at (105.3, 90.8)
- H1: footprint MountingHole:MountingHole_3.2mm_M3_ISO7380 -> MountingHole:MountingHole_3.2mm_M3_ISO14580
- TP1: moved to B.Cu
- moved C9 15.0 mm to (119.5, 90.6)
- moved C7 1.50 mm to (103.0, 90.2)
- moved C8 1.50 mm to (104.5, 90.2)
Connections:
- J1 pad 2: /Rx- -> /_Rx-
- J1 pad 3: /Rx+ -> /_Rx+
- J1 pad 4: /Tx- -> /_Tx-
- J1 pad 5: /Tx+ -> /_Tx+
Routing:
- net /Rx+: track 22.5 -> 5.68 mm
- net /_Rx+: track 0.00 -> 15.7 mm
- net /Rx-: track 21.3 -> 6.70 mm
- net /_Rx-: track 0.00 -> 13.5 mm
- net /Tx-: track 23.3 -> 16.7 mm
- net /Tx+: track 22.5 -> 16.9 mm
- net /_Tx-: track 0.00 -> 5.51 mm
- net GND: track 56.2 -> 61.1 mm, vias 18 -> 26
- net /_Tx+: track 0.00 -> 4.43 mm
- net /VDDA_18: track 25.1 -> 23.8 mm
- net /3V3: track 70.6 -> 71.6 mm
- added copper zone on F.Cu, net GND
Other:
- board text added: "Rev 1 ."
- board text added: "by ElectroMan"

Commit message: As ordered with OSHpark
Parts:
- added C13: 10u, Capacitor_SMD:C_0603_1608Metric_Pad1.08x0.95mm_HandSolder, F.Cu at (117.1, 77.0)
- added C14: 1u, Capacitor_SMD:C_0603_1608Metric_Pad1.08x0.95mm_HandSolder, F.Cu at (114.6, 77.0)
- added C15: 100n, Capacitor_SMD:C_0603_1608Metric_Pad1.08x0.95mm_HandSolder, F.Cu at (112.1, 77.0)
- added TP2: GND, TestPoint:TestPoint_THTPad_D2.5mm_Drill1.2mm, F.Cu at (133.9, 77.2)
- TP1: footprint TestPoint:TestPoint_THTPad_D1.0mm_Drill0.5mm -> TestPoint:TestPoint_THTPad_D2.5mm_Drill1.2mm
- moved REF** 1.90 mm to (121.3, 91.1)
- moved J1 1.00 mm to (131.5, 88.8)
- moved TP1 0.50 mm to (131.0, 77.2)
Routing:
- net GND: track 61.1 -> 67.8 mm, vias 26 -> 31
- net /_Rx+: track 15.7 -> 14.7 mm
- net /_Tx-: track 5.51 -> 6.51 mm
- net /_Tx+: track 4.43 -> 5.43 mm
- net /_Rx-: track 13.5 -> 12.5 mm
Other:
- board text added: "12V"
- board text added: "GND"
