File: Interface.kicad_sch (KiCad schematic)
At the start: 19 parts, among them IC1 PI6CG18201ZDIEX, J1 Bus_PCI_Express_x1, J2 Conn_01x07_MountingPin, U1 AMS1117-1.8, Y1 Crystal

Commit message: Add few details
Parts:
- C3, C4, C7: now not fitted
- J1: value Bus_PCI_Express_x1 -> PCI_Express_x1 female connector; Partnr (none) -> PCIE-036-02-F-D-TH
Connections:
- net 3V3: now also J1.A11 (~{PERST}), J1.B10 (3.3Vaux), J1.B11 (~{WAKE})
- net GND: now also IC1.23 (SS_SEL_TRI)
- net VDDO_18: now also IC1.22 (PD#)
- no-connect marks 16 -> 17
Other:
- note added: "PCI Express Wikipedia"
- note added: "PCIE FOR HACKERS: LINK ANATOMY"
- note added: "PCIe Hardware Design Guide"
Changed lines of the file:
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@@
 (kicad_sch (version 20230121) (generator eeschema)
   (paper "A4")
+  (junction (at 240.03 40.64) (diameter 0) (color 0 0 0 0)
+  )
+  (junction (at 242.57 40.64) (diameter 0) (color 0 0 0 0)
+  )
   (junction (at 63.5 72.39) (diameter 0) (color 0 0 0 0)
   )
@@
   (junction (at 52.07 53.34) (diameter 0) (color 0 0 0 0)
   )
+  (junction (at 124.46 114.3) (diameter 0) (color 0 0 0 0)
+  )
   (junction (at 63.5 34.29) (diameter 0) (color 0 0 0 0)
   )
@@
   (junction (at 96.52 152.4) (diameter 0) (color 0 0 0 0)
   )
+  (junction (at 257.81 63.5) (diameter 0) (color 0 0 0 0)
+  )
   (junction (at 144.78 180.34) (diameter 0) (color 0 0 0 0)
   )
@@
   )
   (junction (at 62.23 144.78) (diameter 0) (color 0 0 0 0)
+  )
+  (junction (at 116.84 116.84) (diameter 0) (color 0 0 0 0)
   )
   (junction (at 111.76 116.84) (diameter 0) (color 0 0 0 0)
@@
   (no_connect (at 255.27 71.12))
   (no_connect (at 255.27 76.2))
+  (no_connect (at 224.79 73.66))
   (no_connect (at 255.27 73.66))
-  (no_connect (at 240.03 48.26))
+  (no_connect (at 224.79 71.12))
   (no_connect (at 99.06 149.86))
   (no_connect (at 224.79 58.42))
@@
     (stroke (width 0) (type default))
   )
+  (wire (pts (xy 255.27 63.5) (xy 257.81 63.5))
+    (stroke (width 0) (type default))
+  )
   (wire (pts (xy 223.52 128.27) (xy 236.22 128.27))
     (stroke (width 0) (type default))
@@
     (stroke (width 0) (type default))
   )
+  (wire (pts (xy 116.84 116.84) (xy 116.84 119.38))
+    (stroke (width 0) (type default))
+  )
   (wire (pts (xy 52.07 67.31) (xy 52.07 72.39))
     (stroke (width 0) (type default))
@@
     (stroke (width 0) (type default))
   )
-  (wire (pts (xy 121.92 116.84) (xy 114.3 116.84))
+  (wire (pts (xy 121.92 116.84) (xy 116.84 116.84))
+    (stroke (width 0) (type default))
+  )
+  (wire (pts (xy 257.81 40.64) (xy 242.57 40.64))
     (stroke (width 0) (type default))
   )
@@
     (stroke (width 0) (type default))
   )
+  (wire (pts (xy 119.38 114.3) (xy 119.38 119.38))
+    (stroke (width 0) (type default))
+  )
+  (wire (pts (xy 255.27 66.04) (xy 257.81 66.04))
+    (stroke (width 0) (type default))
+  )
   (wire (pts (xy 223.52 120.65) (xy 236.22 120.65))
     (stroke (width 0) (type default))
@@
     (stroke (width 0) (type default))
   )
+  (wire (pts (xy 116.84 116.84) (xy 114.3 116.84))
+    (stroke (width 0) (type default))
+  )
   (wire (pts (xy 96.52 152.4) (xy 96.52 154.94))
     (stroke (width 0) (type default))
@@
     (stroke (width 0) (type default))
   )
+  (wire (pts (xy 257.81 63.5) (xy 257.81 40.64))
+    (stroke (width 0) (type default))
+  )
   (wire (pts (xy 139.7 147.32) (xy 156.21 147.32))
     (stroke (width 0) (type default))
@@
     (stroke (width 0) (type default))
   )
-  (wire (pts (xy 236.22 40.64) (xy 242.57 40.64))
+  (wire (pts (xy 236.22 40.64) (xy 240.03 40.64))
     (stroke (width 0) (type default))
   )
@@
     (stroke (width 0) (type default))
   )
+  (wire (pts (xy 119.38 114.3) (xy 124.46 114.3))
+    (stroke (width 0) (type default))
+  )
+  (wire (pts (xy 257.81 66.04) (xy 257.81 63.5))
+    (stroke (width 0) (type default))
+  )
   (wire (pts (xy 223.52 123.19) (xy 236.22 123.19))
     (stroke (width 0) (type default))
@@
     (stroke (width 0) (type default))
   )
+  (wire (pts (xy 240.03 40.64) (xy 240.03 48.26))
+    (stroke (width 0) (type default))
+  )
   (wire (pts (xy 81.28 133.35) (xy 62.23 133.35))
     (stroke (width 0) (type default))
@@
     (stroke (width 0) (type default))
   )
+  (wire (pts (xy 240.03 40.64) (xy 242.57 40.64))
+    (stroke (width 0) (type default))
+  )
   (wire (pts (xy 93.98 147.32) (xy 93.98 180.34))
     (stroke (width 0) (type default))
@@
   (wire (pts (xy 99.06 152.4) (xy 96.52 152.4))
     (stroke (width 0) (type default))
+  )
+  (text "PCIE FOR HACKERS: LINK ANATOMY" (at 212.09 170.18 0)
+    (effects (font (size 1.27 1.27)) (justify left bottom) (href "https://hackaday.com/2023/03/23/pcie-for-hackers-link-anatomy/"))
+  )
+  (text "PCI Express Wikipedia" (at 212.09 180.34 0)
+    (effects (font (size 1.27 1.27)) (justify left bottom) (href "https://en.wikipedia.org/wiki/PCI_Express"))
+  )
+  (text "PCIe Hardware Design Guide" (at 212.09 175.26 0)
+    (effects (font (size 1.27 1.27)) (justify left bottom) (href "https://blog.mbedded.ninja/electronics/communication-protocols/pci-express-pcie/pcie-hardware-design-guide/"))
   )
   (label "VDDO_18" (at 88.9 53.34 180) (fields_autoplaced)
@@
   )
   (symbol (lib_id "Device:C") (at 63.5 38.1 0) (mirror y) (unit 1)
-    (in_bom yes) (on_board yes) (dnp no) (fields_autoplaced)
+    (in_bom yes) (on_board yes) (dnp yes) (fields_autoplaced)
     (property "Reference" "C4" (at 67.31 36.83 0)
       (effects (font (size 1.27 1.27)) (justify right))
@@
       (effects (font (size 1.27 1.27)) hide)
     )
+    (property "Name" "" (at 63.5 38.1 0)
+      (effects (font (size 1.27 1.27)) hide)
+    )
+    (property "Partnr" "" (at 63.5 38.1 0)
+      (effects (font (size 1.27 1.27)) hide)
+    )
     (pin "1")
     (pin "2")
@@
   )
   (symbol (lib_id "Device:C") (at 63.5 57.15 0) (mirror y) (unit 1)
-    (in_bom yes) (on_board yes) (dnp no) (fields_autoplaced)
+    (in_bom yes) (on_board yes) (dnp yes) (fields_autoplaced)
     (property "Reference" "C3" (at 67.31 55.88 0)
       (effects (font (size 1.27 1.27)) (justify right))
@@
     )
     (property "Datasheet" "~" (at 63.5 57.15 0)
+      (effects (font (size 1.27 1.27)) hide)
+    )
+    (property "Name" "" (at 63.5 57.15 0)
+      (effects (font (size 1.27 1.27)) hide)
+    )
+    (property "Partnr" "" (at 63.5 57.15 0)
       (effects (font (size 1.27 1.27)) hide)
     )
@@
       (effects (font (size 1.27 1.27)) (justify left))
     )
-    (property "Value" "Bus_PCI_Express_x1" (at 242.2241 97.79 0)
+    (property "Value" "PCI_Express_x1 female connector" (at 242.2241 97.79 0)
       (effects (font (size 1.27 1.27)) (justify left))
     )
@@
       (effects (font (size 1.27 1.27)) hide)
     )
-    (property "Datasheet" "http://www.ritrontek.com/uploadfile/2016/1026/20161026105231124.pdf#page=63" (at 233.68 92.71 0)
+    (property "Datasheet" "https://www.mouser.dk/datasheet/2/527/pcie-2854633.pdf" (at 233.68 92.71 0)
+      (effects (font (size 1.27 1.27)) hide)
+    )
+    (property "Name" "" (at 240.03 73.66 0)
+      (effects (font (size 1.27 1.27)) hide)
+    )
+    (property "Partnr" "PCIE-036-02-F-D-TH" (at 240.03 73.66 0)
       (effects (font (size 1.27 1.27)) hide)
     )
@@
   )
   (symbol (lib_id "Device:C") (at 63.5 76.2 0) (mirror y) (unit 1)
-    (in_bom yes) (on_board yes) (dnp no) (fields_autoplaced)
+    (in_bom yes) (on_board yes) (dnp yes) (fields_autoplaced)
     (property "Reference" "C7" (at 67.31 74.93 0)
       (effects (font (size 1.27 1.27)) (justify right))
@@
       (effects (font (size 1.27 1.27)) hide)
     )
+    (property "Name" "" (at 63.5 76.2 0)
+      (effects (font (size 1.27 1.27)) hide)
+    )
+    (property "Partnr" "" (at 63.5 76.2 0)
+      (effects (font (size 1.27 1.27)) hide)
+    )

Commit message: Layout
Parts:
- added C10: 100n, Capacitor_SMD:C_0603_1608Metric_Pad1.08x0.95mm_HandSolder, symbol Device:C
- C1: renamed from C4; footprint (none) -> Capacitor_SMD:C_0603_1608Metric_Pad1.08x0.95mm_HandSolder
- C11, C7, C8, C9: footprint (none) -> Capacitor_SMD:C_0603_1608Metric_Pad1.08x0.95mm_HandSolder
- C12: renamed from C10; footprint (none) -> Capacitor_SMD:C_0603_1608Metric_Pad1.08x0.95mm_HandSolder
- C2: renamed from C5; footprint (none) -> Capacitor_SMD:C_0603_1608Metric_Pad1.08x0.95mm_HandSolder
- C3: renamed from C6; footprint (none) -> Capacitor_SMD:C_0603_1608Metric_Pad1.08x0.95mm_HandSolder
- C4: renamed from C3; footprint (none) -> Capacitor_SMD:C_0603_1608Metric_Pad1.08x0.95mm_HandSolder
- C5: renamed from C2; footprint (none) -> Capacitor_SMD:C_0603_1608Metric_Pad1.08x0.95mm_HandSolder
- C6: renamed from C1; footprint (none) -> Capacitor_SMD:C_0603_1608Metric_Pad1.08x0.95mm_HandSolder
- J2: renamed from J1; footprint PCIE-036-02-F-D-TH:PCIE03602FDTH -> Kharars-KiCAD-lib:PCIE03602FDTH
- R1, R2, R3: footprint (none) -> Resistor_SMD:R_0603_1608Metric_Pad0.98x0.95mm_HandSolder
- Y1: value Crystal -> 25MHz; footprint (none) -> Crystal:Crystal_SMD_SeikoEpson_TSX3225-4Pin_3.2x2.5mm_HandSoldering; symbol Device:Crystal -> Device:Crystal_GND24; Manufacturer_Name (none) -> Epson Timing; Manufacturer_Part_Number (none) -> TSX-3225 25.0000MF20X-AJ; Mouser Part Number (none) -> 732-TSX-32525MF2X-AJ
- renumbered J2 to J1
Connections:
- net VDD33 is gone; now on net 3V3: U1.3 (VI)
- net 3V3: now also C10.1
- net GND: now also Y1.2, Y1.4, C10.2
- net at C12.1, IC1.2 (XTAL_OUT): now also Y1.3; no longer Y1.2
Other:
- note added: "OSHpark 2 Layer 2oz 0.8mm Service"
- moved on the sheet: C1, C11, C12, C2, C3, C4, C5, C6, C7, C8, C9, IC1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

Commit message: Continue layout
Parts:
- added H1, H2: MountingHole, MountingHole:MountingHole_3.2mm_M3_ISO7380, symbol Mechanical:MountingHole
- added J1: Conn_01x07_MountingPin, Connector_Molex:Molex_PicoBlade_53047-0710_1x07_P1.25mm_Vertical, symbol Connector_Generic:Conn_01x07
- added TP1: 12V, TestPoint:TestPoint_THTPad_D1.0mm_Drill0.5mm, symbol Connector:TestPoint
- J3: renamed from J1; footprint Connector_Molex:Molex_PicoBlade_53047-0710_1x07_P1.25mm_Vertical -> Connector_Molex:Molex_PicoBlade_53048-0710_1x07_P1.25mm_Horizontal
Connections:
- net 3V3: now also J1.1 (Pin_1)
- net GND: now also J1.6 (Pin_6), J1.7 (Pin_7)
- net Rx+: now also J1.3 (Pin_3)
- net Rx-: now also J1.2 (Pin_2)
- net Tx+: now also J1.5 (Pin_5)
- net Tx-: now also J1.4 (Pin_4)
- net 12V: now reaches J2.A2 (+12V), J2.A3 (+12V), J2.B1 (+12V), J2.B2 (+12V), J2.B3 (+12V)
- net 12V: now also TP1.1
- no-connect marks 17 -> 16

Commit message: Layout finished
Parts:
- removed H2: MountingHole, MountingHole:MountingHole_3.2mm_M3_ISO7380, symbol Mechanical:MountingHole
- removed J3: Conn_01x07_MountingPin, Connector_Molex:Molex_PicoBlade_53048-0710_1x07_P1.25mm_Horizontal, symbol Connector_Generic:Conn_01x07
- added R4, R5, R6, R7: 0, Resistor_SMD:R_0402_1005Metric_Pad0.72x0.64mm_HandSolder, symbol Device:R
- H1: footprint MountingHole:MountingHole_3.2mm_M3_ISO7380 -> MountingHole:MountingHole_3.2mm_M3_ISO14580; now in the parts list
Connections:
- net Rx+: now also R5.1; no longer J1.3 (Pin_3)
- net Rx-: now also R4.1; no longer J1.2 (Pin_2)
- net Tx+: now also R7.1; no longer J1.5 (Pin_5)
- net Tx-: now also R6.1; no longer J1.4 (Pin_4)
- new net _Rx+: J1.3 (Pin_3), R5.2
- new net _Rx-: J1.2 (Pin_2), R4.2
- new net _Tx+: J1.5 (Pin_5), R7.2
- new net _Tx-: J1.4 (Pin_4), R6.2
Other:
- moved on the sheet: J1, J2, TP1

Commit message: As ordered with OSHpark
Parts:
- added C13: 10u, Capacitor_SMD:C_0603_1608Metric_Pad1.08x0.95mm_HandSolder, symbol Device:C
- added C14: 1u, Capacitor_SMD:C_0603_1608Metric_Pad1.08x0.95mm_HandSolder, symbol Device:C
- added C15: 100n, Capacitor_SMD:C_0603_1608Metric_Pad1.08x0.95mm_HandSolder, symbol Device:C
- added TP2: GND, TestPoint:TestPoint_THTPad_D2.5mm_Drill1.2mm, symbol Connector:TestPoint
- TP1: footprint TestPoint:TestPoint_THTPad_D1.0mm_Drill0.5mm -> TestPoint:TestPoint_THTPad_D2.5mm_Drill1.2mm
Connections:
- net 12V: now also C13.1, C14.1, C15.1
- net GND: now also C13.2, C14.2, C15.2, TP2.1
